File: Version 1.1 PCB/BLDC_Version1_1_0.kicad_pcb (KiCad board)
At the start: 4 copper layers, 80 x 80 mm, 124 parts, among them CN1 DB910-7.62-3P, CN2 XT60PW-M, CN3 SM06B-GHS-TB(LF)(SN), CN4 SM03B-GHS-TB(LF)(SN), J1 USB_C_Receptacle_USB2.0_14P, Q1 N_FET_ISC0602NLS, Q2 N_FET_ISC0602NLS, Q3 SI7129DN-T1-GE3, Q4 N_FET_ISC0602NLS, Q5 N_FET_ISC0602NLS, Q6 N_FET_ISC0602NLS, Q7 N_FET_ISC0602NLS, SW1 SW_MEC_5E, SW2 SW_MEC_5E, U1 ESP32-S3-WROOM-1, U10 SRV05-4-HXY, U11 SRV05-4-HXY, U13 SRV05-4-HXY, U14 SRV05-4-HXY, U2 AP7363-33D-13, U3 TMC6200-TA-T, U4 TPS5430DDAR, U7 8x Male Headers, U9 Male Headers

Commit message: Minor changes
Parts:
- added G***: LOGO, Project_BLDC_Foorprint_Library:Cat, F.Cu at (124.6, 101.4)
- C10: footprint Capacitor_SMD:C_0805_2012Metric_Pad1.18x1.45mm_HandSolder -> easyeda2kicad:CAP-SMD_BD6.3-L6.6-W6.6-FD
- Q1, Q2, Q4, Q5, Q6, Q7: footprint Package_SON:Infineon_PG-TDSON-8_6.15x5.15mm -> Project_BLDC_Foorprint_Library:Infineon_PG-TDSON-8_6.15x5.15mm
- moved C3 9.37 mm to (124.3, 125.3), turned to 90 degrees
- moved 5V 3.20 mm to (120.9, 126.5)
- moved C10 1.78 mm to (123.0, 132.6)
- moved CN3 0.50 mm to (128.0, 64.0)
- moved CN4 0.50 mm to (139.0, 64.0)
- moved L1 0.50 mm to (129.5, 132.9)
- moved R10 0.40 mm to (134.4, 132.0)
- moved R11 0.40 mm to (134.4, 135.0)
- renumbered JP3 to AMPL, C16 to CU, C19 to CV, C24 to CW, JP4 to DRV, JP1 to I_0, JP2 to I_1
Routing:
- net GPIO37: track 39.3 -> 38.6 mm
Other:
- board text added: "FUSE"
- board text added: "JLCJLCJLCJLC"
